File: Kicad_v2/LED_Eyes2.kicad_sch (KiCad schematic)
At the start: 18 parts, among them J2 Conn_01x03, U202 74LVC1G17

Commit message: w/w w/o Pegelshifter
Parts:
- added J1: Conn_01x03, Connector_Wire:SolderWire-0.5sqmm_1x03_P4.8mm_D0.9mm_OD2.3mm, symbol Connector_Generic:Conn_01x03
Connections:
- net +5V: now also J1.1 (Pin_1)
- net GND: now also J1.3 (Pin_3)
- net at D1.4 (DIN), R205.1: now also J1.2 (Pin_2)
Changed lines of the file:
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@@
   (junction (at 181.61 27.94) (diameter 0) (color 0 0 0 0)
+  )
+  (junction (at 209.55 21.59) (diameter 0) (color 0 0 0 0)
   )
   (junction (at 209.55 99.06) (diameter 0) (color 0 0 0 0)
@@
     (stroke (width 0) (type default))
   )
+  (wire (pts (xy 223.52 34.29) (xy 223.52 21.59))
+    (stroke (width 0) (type default))
+  )
   (wire (pts (xy 91.44 120.65) (xy 91.44 121.92))
     (stroke (width 0) (type default))
@@
     (stroke (width 0) (type default))
   )
+  (wire (pts (xy 223.52 21.59) (xy 209.55 21.59))
+    (stroke (width 0) (type default))
+  )
   (wire (pts (xy 111.76 161.29) (xy 120.65 161.29))
     (stroke (width 0) (type default))
@@
   )
   (wire (pts (xy 186.69 36.83) (xy 186.69 39.37))
+    (stroke (width 0) (type default))
+  )
+  (wire (pts (xy 231.14 34.29) (xy 223.52 34.29))
     (stroke (width 0) (type default))
   )
@@
         (path "/bba1188b-1353-4037-a6bf-904f73edb043"
           (reference "#PWR02") (unit 1)
+        )
+      )
+    )
+  )
+  (symbol (lib_id "power:+5V") (at 231.14 31.75 0) (unit 1)
+    (in_bom yes) (on_board yes) (dnp no) (fields_autoplaced)
+    (property "Reference" "#PWR03" (at 231.14 35.56 0)
+      (effects (font (size 1.27 1.27)) hide)
+    )
+    (property "Value" "+5V" (at 231.14 26.67 0)
+      (effects (font (size 1.27 1.27)))
+    )
+    (property "Footprint" "" (at 231.14 31.75 0)
+      (effects (font (size 1.27 1.27)) hide)
+    )
+    (property "Datasheet" "" (at 231.14 31.75 0)
+      (effects (font (size 1.27 1.27)) hide)
+    )
+    (pin "1")
+    (instances
+      (project "LED_Eyes2"
+        (path "/65dea14e-ac8e-4f1a-8b68-4fede5b3fd7f"
+          (reference "#PWR03") (unit 1)
         )
       )
@@
     )
   )
+  (symbol (lib_id "power:GND") (at 231.14 36.83 0) (unit 1)
+    (in_bom yes) (on_board yes) (dnp no) (fields_autoplaced)
+    (property "Reference" "#PWR04" (at 231.14 43.18 0)
+      (effects (font (size 1.27 1.27)) hide)
+    )
+    (property "Value" "GND" (at 231.14 41.91 0)
+      (effects (font (size 1.27 1.27)))
+    )
+    (property "Footprint" "" (at 231.14 36.83 0)
+      (effects (font (size 1.27 1.27)) hide)
+    )
+    (property "Datasheet" "" (at 231.14 36.83 0)
+      (effects (font (size 1.27 1.27)) hide)
+    )
+    (pin "1")
+    (instances
+      (project "LED_Eyes2"
+        (path "/65dea14e-ac8e-4f1a-8b68-4fede5b3fd7f"
+          (reference "#PWR04") (unit 1)
+        )
+      )
+    )
+  )
   (symbol (lib_id "power:+5V") (at 153.67 119.38 0) (unit 1)
     (in_bom yes) (on_board yes) (dnp no)
@@
         )
       )
+    )
+  )
+  (symbol (lib_id "Connector_Generic:Conn_01x03") (at 236.22 34.29 0) (unit 1)
+    (in_bom yes) (on_board yes) (dnp no)
+    (property "Reference" "J1" (at 238.76 33.02 0)
+      (effects (font (size 1.27 1.27)) (justify left))
+    )
+    (property "Value" "Conn_01x03" (at 238.76 35.56 0)
+      (effects (font (size 1.27 1.27)) (justify left))
+    )
+    (property "Footprint" "Connector_Wire:SolderWire-0.5sqmm_1x03_P4.8mm_D0.9mm_OD2.3mm" (at 266.7 45.72 0)
+      (effects (font (size 1.27 1.27)))
+    )
+    (property "Datasheet" "~" (at 236.22 34.29 0)
+      (effects (font (size 1.27 1.27)) hide)
+    )
+    (pin "1")
+    (pin "2")
+    (pin "3")
+    (instances
+      (project "LED_Eyes2"
+        (path "/65dea14e-ac8e-4f1a-8b68-4fede5b3fd7f"
+          (reference "J1") (unit 1)
+        )
+      )
