File: Kicad_v2/LED_Eyes2.kicad_pcb (KiCad board)
At the start: 2 copper layers, 107.8 x 68.3 mm, 18 parts, among them J2 Conn_01x03, U1 74LVC1G17

Commit message: PCB CU-lines improved
Routing:
- net Net-(D6-DOUT): track 0.00 -> 21.1 mm
- net +5V: track 7.27 -> 18.9 mm
- net Net-(R1-Pad2): track 0.00 -> 3.25 mm
- net Net-(D1-DIN): track 0.00 -> 2.77 mm
- added copper zone on B.Cu, net GND
Changed lines of the file:
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@@
     )
   )
-  (gr_line (start 172 93.9) (end 175.1 93.9)
-    (stroke (width 0.2) (type default)) (layer "F.Cu"))
-  (gr_line (start 167.5 93.9) (end 170.3 93.9)
-    (stroke (width 0.2) (type default)) (layer "F.Cu"))
   (gr_line (start 128.8932 134.6217) (end 129.0752 134.5729)
     (stroke (width 0.1) (type solid)) (layer "Edge.Cuts"))
@@
   (gr_line (start 130.60006 71.7) (end 130.25631 71.6079)
     (stroke (width 0.1) (type solid)) (layer "Edge.Cuts"))
+  (segment (start 137.55 113.45) (end 137.5 113.4) (width 0.2) (layer "F.Cu") (net 1))
+  (segment (start 137.55 133.95) (end 137.55 131.525) (width 0.2) (layer "F.Cu") (net 1))
+  (segment (start 146.55 124.95) (end 146.55 122.525) (width 0.2) (layer "F.Cu") (net 1))
+  (segment (start 137.55 131.525) (end 137.525 131.5) (width 0.2) (layer "F.Cu") (net 1))
+  (segment (start 128.55 122.775) (end 128.625 122.7) (width 0.2) (layer "F.Cu") (net 1))
+  (segment (start 137.55 115.95) (end 137.55 113.45) (width 0.2) (layer "F.Cu") (net 1))
+  (segment (start 162.55 91.2125) (end 162.5625 91.2) (width 0.2) (layer "F.Cu") (net 1))
+  (segment (start 137.55 124.95) (end 137.55 122.875) (width 0.2) (layer "F.Cu") (net 1))
+  (segment (start 137.55 122.875) (end 137.725 122.7) (width 0.2) (layer "F.Cu") (net 1))
+  (segment (start 146.55 122.525) (end 146.525 122.5) (width 0.2) (layer "F.Cu") (net 1))
+  (segment (start 162.55 93.85) (end 162.55 91.2125) (width 0.2) (layer "F.Cu") (net 1))
+  (segment (start 128.55 124.95) (end 128.55 122.775) (width 0.2) (layer "F.Cu") (net 1))
   (segment (start 112.55 93.85) (end 112.55 91.575) (width 0.2) (layer "F.Cu") (net 1))
-  (segment (start 137.55 133.95) (end 137.55 131.525) (width 0.2) (layer "F.Cu") (net 1))
   (segment (start 112.55 91.575) (end 112.625 91.5) (width 0.2) (layer "F.Cu") (net 1))
-  (segment (start 146.55 122.525) (end 146.525 122.5) (width 0.2) (layer "F.Cu") (net 1))
-  (segment (start 146.55 124.95) (end 146.55 122.525) (width 0.2) (layer "F.Cu") (net 1))
-  (segment (start 139.6 131.5) (end 141.1 131.5) (width 0.2) (layer "F.Cu") (net 2))
-  (segment (start 178.3 97.6) (end 176.65 97.6) (width 0.2) (layer "F.Cu") (net 2))
-  (segment (start 139.575 113.4) (end 141.4 113.4) (width 0.2) (layer "F.Cu") (net 2))
+  (segment (start 175.1 97.6) (end 175.1 95.8) (width 0.2) (layer "F.Cu") (net 1))
+  (segment (start 142.45 119.25) (end 144.55 119.25) (width 0.2) (layer "F.Cu") (net 2))
+  (segment (start 144.15 128.25) (end 144.3 128.4) (width 0.2) (layer "F.Cu") (net 2))
   (segment (start 178.5 93.9) (end 179 94.4) (width 0.2) (layer "F.Cu") (net 2))
+  (segment (start 151.4 128.3) (end 151.45 128.25) (width 0.2) (layer "F.Cu") (net 2))
   (segment (start 177.375 95.8) (end 178.5 95.8) (width 0.2) (layer "F.Cu") (net 2))
+  (segment (start 133.45 128.25) (end 131.55 128.25) (width 0.2) (layer "F.Cu") (net 2))
   (segment (start 167.5 97.2) (end 167.45 97.15) (width 0.2) (layer "F.Cu") (net 2))
   (segment (start 149.65 128.25) (end 149.6 128.3) (width 0.2) (layer "F.Cu") (net 2))
-  (segment (start 140.35 137.25) (end 142.45 137.25) (width 0.2) (layer "F.Cu") (net 2))
+  (segment (start 144.55 119.25) (end 144.6 119.3) (width 0.2) (layer "F.Cu") (net 2))
   (segment (start 177.375 93.9) (end 178.5 93.9) (width 0.2) (layer "F.Cu") (net 2))
+  (segment (start 144.3 128.4) (end 142.6 128.4) (width 0.2) (layer "F.Cu") (net 2))
+  (segment (start 149.6 128.3) (end 151.4 128.3) (width 0.2) (layer "F.Cu") (net 2))
+  (segment (start 114.7 91.5) (end 116.1 91.5) (width 0.2) (layer "F.Cu") (net 2))
+  (segment (start 139.8 122.7) (end 141.2 122.7) (width 0.2) (layer "F.Cu") (net 2))
+  (segment (start 142.45 137.25) (end 140.35 137.25) (width 0.2) (layer "F.Cu") (net 2))
+  (segment (start 133.4 128.3) (end 133.45 128.25) (width 0.2) (layer "F.Cu") (net 2))
+  (segment (start 176.65 97.6) (end 178.3 97.6) (width 0.2) (layer "F.Cu") (net 2))
+  (segment (start 179 94.4) (end 179 94.9) (width 0.2) (layer "F.Cu") (net 2))
+  (segment (start 167.45 97.15) (end 169.15 97.15) (width 0.2) (layer "F.Cu") (net 2))
+  (segment (start 166.7 91.2) (end 164.6375 91.2) (width 0.2) (layer "F.Cu") (net 2))
+  (segment (start 178.5 95.8) (end 179 95.3) (width 0.2) (layer "F.Cu") (net 2))
+  (segment (start 142.6 128.4) (end 142.45 128.25) (width 0.2) (layer "F.Cu") (net 2))
+  (segment (start 141.2 122.7) (end 141.3 122.8) (width 0.2) (layer "F.Cu") (net 2))
+  (segment (start 141.1 131.5) (end 139.6 131.5) (width 0.2) (layer "F.Cu") (net 2))
+  (segment (start 179 95.3) (end 179 94.9) (width 0.2) (layer "F.Cu") (net 2))
+  (segment (start 119.15 97.15) (end 119.2 97.1) (width 0.2) (layer "F.Cu") (net 2))
+  (segment (start 130.7 122.7) (end 132.3 122.7) (width 0.2) (layer "F.Cu") (net 2))
+  (segment (start 117.45 97.15) (end 119.15 97.15) (width 0.2) (layer "F.Cu") (net 2))
+  (segment (start 139.575 113.4) (end 141.4 113.4) (width 0.2) (layer "F.Cu") (net 2))
+  (segment (start 131.55 128.25) (end 131.5 128.3) (width 0.2) (layer "F.Cu") (net 2))
+  (segment (start 169.15 97.15) (end 169.2 97.2) (width 0.2) (layer "F.Cu") (net 2))
   (segment (start 148.6 122.5) (end 150.3 122.5) (width 0.2) (layer "F.Cu") (net 2))
-  (segment (start 114.7 91.5) (end 116.1 91.5) (width 0.2) (layer "F.Cu") (net 2))
-  (segment (start 133.4 128.3) (end 133.45 128.25) (width 0.2) (layer "F.Cu") (net 2))
-  (segment (start 131.5 128.3) (end 133.4 128.3) (width 0.2) (layer "F.Cu") (net 2))
-  (segment (start 140.3 137.3) (end 140.35 137.25) (width 0.2) (layer "F.Cu") (net 2))
-  (segment (start 151.45 128.25) (end 149.65 128.25) (width 0.2) (layer "F.Cu") (net 2))
-  (segment (start 179 94.4) (end 179 94.9) (width 0.2) (layer "F.Cu") (net 2))
-  (segment (start 141.2 122.7) (end 141.3 122.8) (width 0.2) (layer "F.Cu") (net 2))
-  (segment (start 164.6375 91.2) (end 166.7 91.2) (width 0.2) (layer "F.Cu") (net 2))
-  (segment (start 178.5 95.8) (end 179 95.3) (width 0.2) (layer "F.Cu") (net 2))
-  (segment (start 139.8 122.7) (end 141.2 122.7) (width 0.2) (layer "F.Cu") (net 2))
-  (segment (start 179 95.3) (end 179 94.9) (width 0.2) (layer "F.Cu") (net 2))
-  (segment (start 142.45 119.25) (end 144.55 119.25) (width 0.2) (layer "F.Cu") (net 2))
-  (segment (start 142.6 128.4) (end 142.45 128.25) (width 0.2) (layer "F.Cu") (net 2))
-  (segment (start 169.2 97.2) (end 167.5 97.2) (width 0.2) (layer "F.Cu") (net 2))
-  (segment (start 119.15 97.15) (end 119.2 97.1) (width 0.2) (layer "F.Cu") (net 2))
-  (segment (start 144.55 119.25) (end 144.6 119.3) (width 0.2) (layer "F.Cu") (net 2))
-  (segment (start 130.7 122.7) (end 132.3 122.7) (width 0.2) (layer "F.Cu") (net 2))
-  (segment (start 144.3 128.4) (end 142.6 128.4) (width 0.2) (layer "F.Cu") (net 2))
-  (segment (start 117.45 97.15) (end 119.15 97.15) (width 0.2) (layer "F.Cu") (net 2))
+  (segment (start 140.35 137.25) (end 140.3 137.3) (width 0.2) (layer "F.Cu") (net 2))
   (via (at 131.5 128.3) (size 0.6) (drill 0.3) (layers "F.Cu" "B.Cu") (free) (net 2))
   (via (at 179 94.9) (size 0.6) (drill 0.3) (layers "F.Cu" "B.Cu") (free) (net 2))
@@
   (via (at 116.1 91.5) (size 0.6) (drill 0.3) (layers "F.Cu" "B.Cu") (free) (net 2))
   (via (at 144.6 119.3) (size 0.6) (drill 0.3) (layers "F.Cu" "B.Cu") (free) (net 2))
+  (segment (start 171.85 93.9) (end 175.1 93.9) (width 0.2) (layer "F.Cu") (net 3))
   (segment (start 170.8 98.801104) (end 170.8 102.8) (width 0.2) (layer "F.Cu") (net 4))
   (segment (start 177.375 94.85) (end 174.751104 94.85) (width 0.2) (layer "F.Cu") (net 4))
@@
   (segment (start 162.55 97.15) (end 149.45 97.15) (width 0.2) (layer "F.Cu") (net 6))
   (segment (start 149.45 97.15) (end 146.15 93.85) (width 0.2) (layer "F.Cu") (net 6))
+  (segment (start 167.45 93.85) (end 170.15 93.85) (width 0.2) (layer "F.Cu") (net 7))
+  (segment (start 170.15 93.85) (end 170.2 93.9) (width 0.2) (layer "F.Cu") (net 7))
   (segment (start 131.5 126.6) (end 134.8 126.6) (width 0.2) (layer "F.Cu") (net 8))
   (segment (start 135.4 126) (end 135.4 118.8) (width 0.2) (layer "F.Cu") (net 8))
@@
   (segment (start 139.85 128.25) (end 142.45 130.85) (width 0.2) (layer "F.Cu") (net 10))
   (segment (start 137.55 128.25) (end 139.85 128.25) (width 0.2) (layer "F.Cu") (net 10))
+  (segment (start 143.2 135.6) (end 148.3 130.5) (width 0.2) (layer "F.Cu") (net 11))
+  (segment (start 137.55 137.25) (end 139.2 135.6) (width 0.2) (layer "F.Cu") (net 11))
+  (segment (start 148.3 130.5) (end 148.3 126.9) (width 0.2) (layer "F.Cu") (net 11))
+  (segment (start 148.3 126.9) (end 150.25 124.95) (width 0.2) (layer "F.Cu") (net 11))
+  (segment (start 139.2 135.6) (end 143.2 135.6) (width 0.2) (layer "F.Cu") (net 11))
+  (segment (start 150.25 124.95) (end 151.45 124.95) (width 0.2) (layer "F.Cu") (net 11))
   (zone (net 1) (net_name "+5V") (layer "F.Cu") (hatch edge 0.5)
     (priority 1)
@@
       )
     )
+  )
+  (zone (net 2) (net_name "GND") (layer "B.Cu") (hatch edge 0.5)
+    (connect_pads (clearance 0.5))
+    (min_thickness 0.25) (filled_areas_thickness no)
+    (fill yes (thermal_gap 0.5) (thermal_bridge_width 0.5))
+    (polygon
+      (pts
+        (xy 208.9 66.5)
+        (xy 69.1 65.8)
+        (xy 73.9 147.1)
+        (xy 203.8 146.6)
+        (xy 209.2 63.3)
+      )
+    )

Commit message: w/w w/o Pegelshifter
Parts:
- added J1: Conn_01x03, Connector_Wire:SolderWire-0.5sqmm_1x03_P4.8mm_D0.9mm_OD2.3mm, F.Cu at (159.4, 87.0)
Routing:
- net Net-(D1-DIN): track 2.77 -> 12.0 mm
Changed lines of the file:
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@@
     (property "ki_keywords" "connector")
     (attr exclude_from_pos_files)
-    (fp_text reference "J2" (at -3.2 -1) (layer "F.SilkS")
+    (fp_text reference "J2" (at 13.4 -0.1) (layer "F.SilkS")
         (effects (font (size 1 1) (thickness 0.15)))
     )
-    (fp_text value "Conn_01x03" (at 4.8 2.35) (layer "F.Fab")
+    (fp_text value "Conn_01x03" (at 2.7 4.1) (layer "F.Fab")
         (effects (font (size 1 1) (thickness 0.15)))
     )
@@
     )
   )
+  (footprint "Connector_Wire:SolderWire-0.5sqmm_1x03_P4.8mm_D0.9mm_OD2.3mm" (layer "F.Cu")
+    (at 159.4 87)
+    (descr "Soldered wire connection, for 3 times 0.5 mm² wires, reinforced insulation, conductor diameter 0.9mm, outer diameter 2.3mm, size source Multi-Contact FLEXI-xV 0.5 (https://ec.staubli.com/AcroFiles/Catalogues/TM_Cab-Main-11014119_(en)_hi.pdf), bend radius 3 times outer diameter, generated with kicad-footprint-generator")
+    (tags "connector wire 0.5sqmm")
+    (property "Sheetfile" "LED_Eyes2.kicad_sch")
+    (property "Sheetname" "")
+    (property "ki_description" "Generic connector, single row, 01x03, script generated (kicad-library-utils/schlib/autogen/connector/)")
+    (property "ki_keywords" "connector")
+    (attr exclude_from_pos_files)
+    (fp_text reference "J1" (at 13 0.2) (layer "F.SilkS")
+        (effects (font (size 1 1) (thickness 0.15)))
+    )
+    (fp_text value "Conn_01x03" (at 2.2 -3) (layer "F.Fab")
+        (effects (font (size 1 1) (thickness 0.15)))
+    )
+    (fp_text user "${REFERENCE}" (at 4.8 0) (layer "F.Fab")
+        (effects (font (size 0.58 0.58) (thickness 0.09)))
+    )
+    (fp_line (start -1.9 -1.65) (end -1.9 1.65)
+      (stroke (width 0.05) (type solid)) (layer "F.CrtYd"))
+    (fp_line (start -1.9 1.65) (end 1.9 1.65)
+      (stroke (width 0.05) (type solid)) (layer "F.CrtYd"))
+    (fp_line (start 1.9 -1.65) (end -1.9 -1.65)
+      (stroke (width 0.05) (type solid)) (layer "F.CrtYd"))
+    (fp_line (start 1.9 1.65) (end 1.9 -1.65)
+      (stroke (width 0.05) (type solid)) (layer "F.CrtYd"))
+    (fp_line (start 2.9 -1.65) (end 2.9 1.65)
+      (stroke (width 0.05) (type solid)) (layer "F.CrtYd"))
+    (fp_line (start 2.9 1.65) (end 6.7 1.65)
+      (stroke (width 0.05) (type solid)) (layer "F.CrtYd"))
+    (fp_line (start 6.7 -1.65) (end 2.9 -1.65)
+      (stroke (width 0.05) (type solid)) (layer "F.CrtYd"))
+    (fp_line (start 6.7 1.65) (end 6.7 -1.65)
+      (stroke (width 0.05) (type solid)) (layer "F.CrtYd"))
+    (fp_line (start 7.7 -1.65) (end 7.7 1.65)
+      (stroke (width 0.05) (type solid)) (layer "F.CrtYd"))
+    (fp_line (start 7.7 1.65) (end 11.5 1.65)
+      (stroke (width 0.05) (type solid)) (layer "F.CrtYd"))
+    (fp_line (start 11.5 -1.65) (end 7.7 -1.65)
+      (stroke (width 0.05) (type solid)) (layer "F.CrtYd"))
+    (fp_line (start 11.5 1.65) (end 11.5 -1.65)
+      (stroke (width 0.05) (type solid)) (layer "F.CrtYd"))
+    (fp_circle (center 0 0) (end 1.15 0)
+      (stroke (width 0.1) (type solid)) (fill none) (layer "F.Fab"))
+    (fp_circle (center 4.8 0) (end 5.95 0)
+      (stroke (width 0.1) (type solid)) (fill none) (layer "F.Fab"))
+    (fp_circle (center 9.6 0) (end 10.75 0)
+      (stroke (width 0.1) (type solid)) (fill none) (layer "F.Fab"))
+    (pad "1" thru_hole roundrect (at 0 0) (size 2.3 2.3) (drill 1.1) (layers "*.Cu" "*.Mask") (roundrect_rratio 0.108696)
+      (net 1 "+5V") (pinfunction "Pin_1") (pintype "passive"))
+    (pad "2" thru_hole circle (at 4.8 0) (size 2.3 2.3) (drill 1.1) (layers "*.Cu" "*.Mask")
+      (net 7 "Net-(D1-DIN)") (pinfunction "Pin_2") (pintype "passive"))
+    (pad "3" thru_hole circle (at 9.6 0) (size 2.3 2.3) (drill 1.1) (layers "*.Cu" "*.Mask")
+      (net 2 "GND") (pinfunction "Pin_3") (pintype "passive"))
+    (model "${KICAD6_3DMODEL_DIR}/Connector_Wire.3dshapes/SolderWire-0.5sqmm_1x03_P4.8mm_D0.9mm_OD2.3mm.wrl"
+      (offset (xyz 0 0 0))
+      (scale (xyz 1 1 1))
+      (rotate (xyz 0 0 0))
+    )
+  )
   (footprint "LED_SMD:LED_WS2812B_PLCC4_5.0x5.0mm_P3.2mm" (layer "F.Cu")
     (at 140 126.6)
@@
   (segment (start 162.55 97.15) (end 149.45 97.15) (width 0.2) (layer "F.Cu") (net 6))
   (segment (start 149.45 97.15) (end 146.15 93.85) (width 0.2) (layer "F.Cu") (net 6))
+  (segment (start 167.45 88.45) (end 167.45 93.85) (width 0.2) (layer "F.Cu") (net 7))
+  (segment (start 164.2 87) (end 166 87) (width 0.2) (layer "F.Cu") (net 7))
   (segment (start 167.45 93.85) (end 170.15 93.85) (width 0.2) (layer "F.Cu") (net 7))
   (segment (start 170.15 93.85) (end 170.2 93.9) (width 0.2) (layer "F.Cu") (net 7))
+  (segment (start 166 87) (end 167.45 88.45) (width 0.2) (layer "F.Cu") (net 7))
   (segment (start 131.5 126.6) (end 134.8 126.6) (width 0.2) (layer "F.Cu") (net 8))
   (segment (start 135.4 126) (end 135.4 118.8) (width 0.2) (layer "F.Cu") (net 8))

Commit message: Leiterbahnenbreite
Routing:
- net Net-(J2-Pin_2): track 12.2 -> 12.9 mm
